File: DAC.sch (EAGLE design)
At the start: 119 parts, among them IC1 XHRA-2HPA, IC10 TLE2141ACP, IC2 STF202-22T1G, IC3 ADM1085AKSZ-REEL7, IC4 STM1061N38WX6F, IC5 SN74LVC1G06, IC6 PCM1795DB, IC7 LME49720NA_NOPB, IC8 LME49720NA_NOPB, IC9 LME49720NA_NOPB, J1 USB_B_PTH, U1 S25FL132K, Y1 DSC1001CL2-022.5972, Y2 DSC1001BI1-024.5760, Y3 DSC1001BC1-024.0000

Commit message: Add layout progress
Parts:
- removed C16, C17, C18: 100n, resistor:C-EUC0603K
- removed C26, C28, C29, C32: 10u, resistor:CPOL-EUA/3216-18R
- removed JP2, JP3: (no value), pinhead:PINHD-1X8
- added GND, GPI: (no value), pinhead:PINHD-1X3
- renumbered JP10 to J10, JP12 to J12, JP13 to J13, JP14 to J14, JP15 to J15, JP16 to J16, JP17 to J17, JP18 to J18, JP19 to J19, JP5 to J5, JP6 to J6, JP7 to J7, JP8 to J8, JP9 to J9
Connections:
- net 1V: no longer C16.1, C17.1, C18.1
- net 3.3V: no longer C26.+
- net 5V: no longer C28.+, C29.+, C32.+, JP3.1, JP3.2, JP3.3, JP3.4
- net GND: now also GND.1, GND.2, GND.3; no longer C16.2, C17.2, C18.2, C26.-, C28.-, C29.-, C32.-, JP3.5, JP3.6, JP3.7, JP3.8
- net GPI_0: no longer JP2.1
- net GPI_1: no longer JP2.2
- net GPI_2: no longer JP2.7
- net GPI_3: now also GPI.1; no longer JP2.4
- net GPI_4: now also GPI.2; no longer JP2.5
- net GPI_5: now also GPI.3; no longer JP2.6
- net GPI_6: no longer JP2.3
- net GPI_7: no longer JP2.8
Other:
- moved on the sheet: C15, R11
